File: KiCAD/General_8th_MFB_LPF/General_8th_MFB_LPF.kicad_pcb (KiCad board)
At the start: 2 copper layers, 67.3 x 55.9 mm, 48 parts, among them J1 IN, J2 8TH_OUT, J4 TP_GND, J5 PWR_OUT, J6 PWR_IN, U1 NJM4580, U2 NJM4580, U3 NJM4580

Commit message: PCB Design
Parts:
- removed the J4 at (191.8, 104.1)
- removed the J5 at (175.3, 115.6)
- removed the R4 at (134.0, 92.1)
- added J3: S_PWR_IN, Connector_JST:JST_XH_B2B-XH-A_1x02_P2.50mm_Vertical, F.Cu at (170.1, 116.2)
- added R15: R, Resistor_THT:R_Axial_DIN0207_L6.3mm_D2.5mm_P7.62mm_Horizontal, F.Cu at (146.7, 77.5)
- J1: renamed from J6; value PWR_IN -> D_PWR_IN
- moved J5 62.7 mm to (179.1, 75.6), turned to 270 degrees
- moved JP1 46.4 mm to (181.0, 104.1), turned to 90 degrees
- moved J2 46.0 mm to (179.1, 86.4), turned to 270 degrees
- moved R2 44.5 mm to (178.4, 109.9), turned to 180 degrees
- moved J4 42.6 mm to (158.8, 114.9), turned to 0 degrees
- moved U3 39.4 mm to (135.9, 74.9), turned to 0 degrees
- moved R10 38.1 mm to (130.8, 108.6), turned to 0 degrees
- moved C6 36.2 mm to (133.4, 104.1), turned to 0 degrees
- moved R9 35.0 mm to (141.0, 108.6)
- moved C10 34.9 mm to (128.9, 114.9), turned to 0 degrees
- moved R12 31.2 mm to (132.7, 78.1), turned to 180 degrees
- moved C12 30.7 mm to (125.7, 85.1)
- moved C9 30.6 mm to (150.5, 114.9)
- moved C4 30.1 mm to (162.6, 97.2), turned to 270 degrees
- moved R1 29.2 mm to (163.2, 94.0), turned to 0 degrees
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- renumbered C15 to C1, C16 to C10, C9 to C11, C2 to C12, C5 to C13, C12 to C14, C11 to C15, C6 to C16, C7 to C2, C1 to C3, C14 to C4, C3 to C5, C10 to C6, C8 to C7, C4 to C8, C13 to C9, J1 to J2, J2 to J5, R5 to R1, R16 to R10, R9 to R11, R2 to R12, R10 to R13, R11 to R14, R12 to R16, R14 to R2, R15 to R3, R1 to R4, R6 to R5, R7 to R6, R3 to R7, R13 to R9
Connections:
- C3 pad 1: Net-(C1-Pad1) -> Net-(C3-Pad1)
- C3 pad 2: Net-(C1-Pad2) -> Net-(C3-Pad2)
- C8 pad 1: Net-(C4-Pad1) -> Net-(C8-Pad1)
- C8 pad 2: Net-(C4-Pad2) -> Net-(C8-Pad2)
- J2 pad 1: Net-(J1-Pad1) -> Net-(J2-Pad1)
- R1 pad 2: Net-(R5-Pad2) -> Net-(R1-Pad2)
- R11 pad 2: Net-(C4-Pad1) -> Net-(C8-Pad1)
- R2 pad 2: Net-(R14-Pad2) -> Net-(R2-Pad2)
- R3 pad 1: Net-(R14-Pad2) -> Net-(R2-Pad2)
- R4 pad 1: Net-(C1-Pad1) -> Net-(C3-Pad1)
- R5 pad 1: Net-(C1-Pad2) -> Net-(C3-Pad2)
- R6 pad 2: Net-(C1-Pad1) -> Net-(C3-Pad1)
- R7 pad 1: Net-(C4-Pad1) -> Net-(C8-Pad1)
- R8 pad 1: Net-(C4-Pad2) -> Net-(C8-Pad2)
- U1 pad 1: Net-(JP1-Pad1) -> Net-(R1-Pad2)
- U1 pad 2: Net-(JP1-Pad1) -> Net-(R1-Pad2)
- U1 pad 3: Net-(R14-Pad2) -> Net-(J2-Pad1)
- U1 pad 5: Net-(J1-Pad1) -> Net-(R2-Pad2)
- U1 pad 6: Net-(R5-Pad2) -> Net-(JP1-Pad1)
- U1 pad 7: Net-(R5-Pad2) -> Net-(JP1-Pad1)
- U2 pad 1: Net-(C1-Pad1) -> Net-(C8-Pad1)
- U2 pad 2: Net-(C1-Pad2) -> Net-(C8-Pad2)
- U2 pad 6: Net-(C4-Pad2) -> Net-(C3-Pad2)
- U2 pad 7: Net-(C4-Pad1) -> Net-(C3-Pad1)
Routing:
- added copper zone on B.Cu, net GND
- added copper zone on F.Cu, net GND
Other:
- board text added: "8TH MFB LPF V1.1"
- board text removed: "8TH MFB LPF V1.0"
- board text removed: "D_PWR_IN"
- board text removed: "D_PWR_OUT"
- board text removed: "G"
- board text removed: "GND"
- board text removed: "IN"
- board text removed: "S_PWR_IN"
