File: KiCAD/General_8th_MFB_LPF/General_8th_MFB_LPF.kicad_pcb (KiCad board)
At the start: 2 copper layers, 67.3 x 55.9 mm, 47 parts, among them J1 D_PWR_IN, J2 IN, J3 S_PWR_IN, J4 TP_GND, J5 8TH_OUT, U1 NJM4580, U2 NJM4580, U3 NJM4580

Commit message: Update: PCB Design
Parts:
- added G***: LOGO, myfootprint:Silk_PNPN_Manufactory_600dpi, F.Cu at (166.4, 76.2)
- moved J4 27.4 mm to (179.1, 96.5), turned to 90 degrees
Routing:
- net VCC: track 0.00 -> 107.5 mm
- net VEE: track 0.00 -> 101.5 mm
- net Net-(C7-Pad1): track 0.00 -> 47.5 mm
- net Net-(C16-Pad1): track 0.00 -> 44.0 mm
- net Net-(C15-Pad1): track 0.00 -> 41.3 mm
- net Net-(C11-Pad1): track 0.00 -> 25.2 mm
- net GND: track 0.00 -> 24.9 mm, vias 0 -> 41
- net Net-(C8-Pad2): track 0.00 -> 21.6 mm
- net Net-(C2-Pad1): track 0.00 -> 20.6 mm
- net Net-(J2-Pad1): track 0.00 -> 17.4 mm
- net Net-(C12-Pad1): track 0.00 -> 17.0 mm
- net Net-(C3-Pad1): track 0.00 -> 16.4 mm
- net Net-(JP1-Pad1): track 0.00 -> 14.3 mm
- net Net-(C8-Pad1): track 0.00 -> 11.4 mm
- net Net-(C12-Pad2): track 0.00 -> 11.0 mm
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Other:
- board text added: "G IN"
- board text added: "G OUT"
- board text added: "GND"
- board text added: "VGND"
