File: KiCAD/General_8th_MFB_LPF/General_8th_MFB_LPF.sch (KiCad schematic (older format))
At the start: 47 parts, among them J1 IN, J2 8TH_OUT, J4 TP_GND, J5 PWR_OUT, J6 PWR_IN, U1 NJM4580, U2 NJM4580, U3 NJM4580

Commit message: PCB Design
Parts:
- removed J5: PWR_OUT, Connector_JST:JST_XH_B3B-XH-A_1x03_P2.50mm_Vertical, symbol Connector_Generic:Conn_01x03
- added J3: S_PWR_IN, Connector_JST:JST_XH_B2B-XH-A_1x02_P2.50mm_Vertical, symbol Connector_Generic:Conn_01x02
- J1: renamed from J6; value PWR_IN -> D_PWR_IN
- renumbered C15 to C1, C16 to C10, C9 to C11, C2 to C12, C5 to C13, C12 to C14, C11 to C15, C6 to C16, C7 to C2, C1 to C3, C14 to C4, C3 to C5, C10 to C6, C8 to C7, C4 to C8, C13 to C9, J1 to J2, J2 to J5, R5 to R1, R16 to R10, R9 to R11, R2 to R12, R10 to R13, R11 to R14, R4 to R15, R12 to R16, R14 to R2, R15 to R3, R1 to R4, R6 to R5, R7 to R6, R3 to R7, R13 to R9
Connections:
- net VCC: now also J3.1 (Pin_1)
- net VEE: now also J3.2 (Pin_2)
- net at C3.1, R4.1, R6.2: now also U2.7; no longer U2.1
- net at C3.2, R5.1: now also U2.6 (-); no longer U2.2 (-)
- net at C8.2, R8.1: now also U2.2 (-); no longer U2.6 (-)
- net at C8.1, R11.2, R7.1: now also U2.1; no longer U2.7
- net at U1.6 (-), U1.7: now also JP1.1 (A); no longer R1.2
- net at J2.1 (Pin_1): now also U1.3 (+); no longer U1.5 (+)
- net at R2.2, R3.1: now also U1.5 (+); no longer U1.3 (+)
- net at U1.1, U1.2 (-): now also R1.2; no longer JP1.1 (A)
Other:
- moved on the sheet: C1, C10, C4, C9, D1, D2, J1, JP1, R10, R2, R3, R9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
